File: Radiante-Lite-Gen2/Radiante-Lite-Gen2.kicad_pcb (KiCad board)
At the start: 2 copper layers, 66 x 35 mm, 59 parts, among them J1 USB_C_Receptacle_USB2.0_16P, J2 HDMI_A, J3 Micro_SD_Card_Det_Hirose_DM3AT, J4 Conn_01x03, J5 Conn_02x20_Odd_Even, SW1 SW_Push, SW2 SW_Push, U1 RP2350_80QFN, U2 W25Q128JVS, U3 ADXL345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

Commit message: partially laying out
Parts:
- moved U1 80.3 mm to (122.5, 55.3), turned to 90 degrees
- moved U2 67.9 mm to (108.4, 50.7), turned to 90 degrees

Commit message: trying to not being a lazy fucktard on designing the lite gen 2
Parts:
- added C22: 100n, Capacitor_SMD:C_0402_1005Metric, F.Cu at (119.1, 48.6)
- added C23: 100n, Capacitor_SMD:C_0402_1005Metric, F.Cu at (118.0, 48.6)
- added C24: 100n, Capacitor_SMD:C_0402_1005Metric, F.Cu at (115.9, 54.7)
- moved C10 88.4 mm to (129.3, 55.9)
- moved C6 88.4 mm to (129.4, 54.7)
- moved C9 88.3 mm to (129.3, 57.9)
- moved C5 84.6 mm to (122.0, 48.6), turned to 90 degrees
- moved C3 84.3 mm to (122.3, 61.9), turned to -90 degrees
- moved C8 83.5 mm to (124.3, 61.9), turned to -90 degrees
- moved C11 82.5 mm to (126.3, 48.6), turned to 90 degrees
- moved C7 79.6 mm to (120.3, 61.8), turned to -90 degrees
- moved C12 79.2 mm to (123.0, 48.6), turned to 90 degrees
- moved C4 78.5 mm to (116.2, 49.9), turned to 90 degrees
- moved R1 78.3 mm to (114.6, 50.4)
- moved C1 78.1 mm to (116.3, 52.3), turned to 90 degrees
- moved C2 77.3 mm to (115.4, 52.3), turned to 90 degrees
- moved C13 72.0 mm to (115.9, 57.5), turned to 180 degrees
- moved L1 67.9 mm to (113.5, 52.3), turned to 90 degrees
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Connections:
- C21 pad 2: +3V3 -> +3.3V
- J3 pad 4: +3V3 -> +3.3V
- RN3 pad 5: +3V3 -> +3.3V
- RN3 pad 6: +3V3 -> +3.3V
- RN3 pad 7: +3V3 -> +3.3V
- RN3 pad 8: +3V3 -> +3.3V
- RN4 pad 3: +3V3 -> +3.3V
- RN4 pad 4: +3V3 -> +3.3V
Routing:
- net /DVI_CEC: track 0.00 -> 39.1 mm, vias 0 -> 2
- net /DVI_L0M: track 0.00 -> 34.1 mm, vias 0 -> 2
- net /DVI_CKM: track 0.00 -> 34.1 mm, vias 0 -> 2
- net /DVI_L1M: track 0.00 -> 33.4 mm, vias 0 -> 2
- net /DVI_L1P: track 0.00 -> 33.0 mm, vias 0 -> 2
- net /DVI_CKP: track 0.00 -> 32.9 mm, vias 0 -> 2
- net /DVI_L0P: track 0.00 -> 32.8 mm, vias 0 -> 2
- net /DVI_SCL: track 0.00 -> 30.1 mm, vias 0 -> 2
- net /DVI_SDA: track 0.00 -> 28.3 mm
- net /DVI_L2M: track 0.00 -> 27.3 mm
- net /DVI_L2P: track 0.00 -> 26.7 mm, vias 0 -> 2
- net /DVI_HOTPLUG: track 0.00 -> 25.4 mm, vias 0 -> 2
- net Net-(J2-SDA): track 0.00 -> 10.8 mm, vias 0 -> 2
- net Net-(J2-SCL): track 0.00 -> 10.1 mm, vias 0 -> 2
- net Net-(J2-D2+): track 0.00 -> 3.75 mm
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- added copper zone on F.Cu, net +1V1
- added copper zone on F.Cu, net +3.3V
- added copper zone on F.Cu, net /VREG_LX
