File: Radiante-Lite-Gen2/Radiante-Lite-Gen2.kicad_sch (KiCad schematic)
At the start: 51 parts, among them J1 USB_C_Receptacle_USB2.0_16P, J2 HDMI_A, J3 Micro_SD_Card_Det_Hirose_DM3AT, SW1 SW_Push, SW2 SW_Push, U1 RP2350_80QFN, U2 W25Q128JVS, U3 ADXL345, U4 MIC5205-3.3YM5, U5 TXS0102YZP, Y1 12MHz

Commit message: add the pcb
Parts:
- added D3: EMERALD, LED_SMD:LED_0402_1005Metric, symbol Device:LED
- added H1, H2, H3, H4: MountingHole_Pad, MountingHole:MountingHole_2.2mm_M2_Pad_TopBottom, symbol Mechanical:MountingHole_Pad
- added J4: Conn_01x03, Connector_JST:JST_SH_BM03B-SRSS-TB_1x03-1MP_P1.00mm_Vertical, symbol Connector_Generic:Conn_01x03
- added J5: Conn_02x20_Odd_Even, Connector_PinHeader_2.54mm:PinHeader_2x20_P2.54mm_Vertical, symbol Connector_Generic:Conn_02x20_Odd_Even
- added R13: 330, Resistor_SMD:R_0402_1005Metric, symbol Device:R
- J1: footprint Connector_USB:USB_C_Receptacle_GCT_USB4110 -> Connector_USB:USB_C_Receptacle_GCT_USB4105-xx-A_16P_TopMnt_Horizontal
- L1: footprint RP2350_60QFN_minimal:L_pol_2016 -> RP2350_80QFN_minimal:L_pol_2016
Connections:
- net +3.3V: now also J5.8 (Pin_8)
- net GND: now also U1.81 (GND), D3.1 (K), H1.1, H2.1, H3.1, H4.1, J4.2 (Pin_2), J5.15 (Pin_15), J5.16 (Pin_16), J5.25 (Pin_25), J5.26 (Pin_26), J5.35 (Pin_35), J5.36 (Pin_36), J5.5 (Pin_5), J5.6 (Pin_6)
- net GYRO_SCL: now also U1.28 (GPIO27)
- net GYRO_SDA: now also U1.27 (GPIO26)
- net VBUS: now also J5.2 (Pin_2)
- net VSYS: now also J5.4 (Pin_4)
- net P4: now reaches U1.1 (GPIO4)
- net P4: now also J5.11 (Pin_11)
- net P5: now reaches U1.2 (GPIO5)
- net P5: now also J5.13 (Pin_13)
- net P6: now reaches U1.3 (GPIO6)
- net P6: now also J5.17 (Pin_17)
- net DBG_CLK: now reaches U1.33 (SWCLK)
- net DBG_CLK: now also J4.3 (Pin_3)
- net DBG_DAT: now reaches U1.34 (SWD)
- net DBG_DAT: now also J4.1 (Pin_1)
- net P28: now reaches U1.36 (GPIO28)
- net P28: now also J5.21 (Pin_21), R13.1
- net P29: now reaches U1.37 (GPIO29)
- net P29: now also J5.23 (Pin_23)
- net P30: now reaches U1.38 (GPIO30)
- net P30: now also J5.27 (Pin_27)
- net P31: now reaches U1.39 (GPIO31)
- net P31: now also J5.29 (Pin_29)
- net P7: now reaches U1.4 (GPIO7)
- net P7: now also J5.19 (Pin_19)
- net P32: now reaches U1.40 (GPIO32)
- net P32: now also J5.31 (Pin_31)
- net P33: now reaches U1.42 (GPIO33)
- net P33: now also J5.33 (Pin_33)
- net P34: now reaches U1.43 (GPIO34)
- net P34: now also J5.37 (Pin_37)
- net P35: now reaches U1.44 (GPIO35)
- net P35: now also J5.39 (Pin_39)
- net P36: now reaches U1.45 (GPIO36)
- net P36: now also J5.40 (Pin_40)
- net P37: now reaches U1.46 (GPIO37)
- net P37: now also J5.38 (Pin_38)
- net P38: now reaches U1.47 (GPIO38)
- net P38: now also J5.34 (Pin_34)
- net P39: now reaches U1.48 (GPIO39)
- net P39: now also J5.32 (Pin_32)
- net P40: now reaches U1.49 (GPIO40_ADC0)
- net P40: now also J5.30 (Pin_30)
- net P41: now reaches U1.52 (GPIO41_ADC1)
- net P41: now also J5.28 (Pin_28)
- net P42: now reaches U1.53 (GPIO42_ADC2)
- net P42: now also J5.24 (Pin_24)
- net P43: now reaches U1.54 (GPIO43_ADC3)
- net P43: now also J5.22 (Pin_22)
- net P44: now reaches U1.55 (GPIO44_ADC4)
- net P44: now also J5.20 (Pin_20)
- net P45: now reaches U1.56 (GPIO45_ADC5)
- net P45: now also J5.18 (Pin_18)
- net P46: now reaches U1.57 (GPIO46_ADC6)
- net P46: now also J5.14 (Pin_14)
- net P47: now reaches U1.58 (GPIO47_ADC7)
- net P47: now also J5.12 (Pin_12)
- net P0: now reaches U1.77 (GPIO0)
- net P0: now also J5.1 (Pin_1)
- net P1: now reaches U1.78 (GPIO1)
- net P1: now also J5.3 (Pin_3)
- net P2: now reaches U1.79 (GPIO2)
- net P2: now also J5.7 (Pin_7)
- net P3: now reaches U1.80 (GPIO3)
- net P3: now also J5.9 (Pin_9)
- new net: D3.2 (A), R13.2
- no-connect marks 9 -> 10

Commit message: trying to not being a lazy fucktard on designing the lite gen 2
Parts:
- added C22, C23, C24: 100n, Capacitor_SMD:C_0402_1005Metric, symbol Device:C
Connections:
- net +3V3 is gone; now on net +3.3V: C21.2, J3.4 (VDD), RN3.5 (R4.2), RN3.6 (R3.2), RN3.7 (R2.2), RN3.8 (R1.2), RN4.3 (R2.2), RN4.4 (R1.2)
- net +3.3V: now also C22.1, C23.1, C24.1
- net GND: now also C22.2, C23.2, C24.2
