File: Radianite-ProjectLemonIrvine/Radianite-ProjectLemonIrvine.kicad_pcb (KiCad board)
At the start: 4 copper layers, 85 x 56 mm, 177 parts, among them J1 FAN, J2 Micro_SD_Card_Det2, J3 Conn_02x20_Odd_Even, J4 RJ45_Abracon_ARJP11A-MASA-B-A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, J5 USB_C_Receptacle_USB2.0_16P, J6 USB_A_Stacked, J7 USB_A_Stacked, J8 AudioJack4, J9 HDMI_A, SW1 434133025816, SW2 434133025816, U7 CH340N, Y1 40MHz, Y2 40MHz

Commit message: upstream sync
Parts:
- moved C48 28.3 mm to (95.6, 49.7)
- moved C49 28.3 mm to (95.6, 51.6)
- moved C50 28.3 mm to (95.6, 53.5)
- moved C51 28.3 mm to (95.6, 55.5)
- moved C52 28.3 mm to (95.6, 57.5)
- moved C53 28.3 mm to (95.6, 59.4)
- moved C54 28.3 mm to (95.6, 61.3)
- moved C30 28.3 mm to (93.2, 50.1)
- moved C31 28.3 mm to (93.2, 51.1)
- moved C32 28.3 mm to (93.2, 52.1)
- moved C33 28.3 mm to (97.0, 49.2)
- moved C34 28.3 mm to (97.0, 53.1)
- moved C35 28.3 mm to (97.0, 52.1)
- moved C36 28.3 mm to (97.0, 51.1)
- moved C37 28.3 mm to (97.0, 59.0)
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Routing:
- net VRAM: track 48.9 -> 11.1 mm, vias 28 -> 10
- net /Memory/SDQ1: track 4.38 -> 0.04 mm
- net /Memory/SDQ6: track 0.00 -> 0.42 mm, vias 0 -> 1

Commit message: woopsies, wrong sd card direction
Parts:
- added ?: , , F.Cu at (119.9, 47.4)
- added ?: , , F.Cu at (119.9, 48.5)
- added ?: , , F.Cu at (119.9, 50.5)
- added ?: , , F.Cu at (119.9, 49.5)
- added C34: 100n, Capacitor_SMD:C_0402_1005Metric, B.Cu at (119.5, 48.5)
- added C35: 100n, Capacitor_SMD:C_0402_1005Metric, B.Cu at (119.5, 49.5)
- added C36: 100n, Capacitor_SMD:C_0402_1005Metric, B.Cu at (119.5, 50.5)
- added C55: 100n, Capacitor_SMD:C_0402_1005Metric, B.Cu at (119.5, 47.4)
- C39, C40, C41, C42, C43, C44: moved to F.Cu
- C58, C59, C60, R11: moved to B.Cu
- moved R11 77.0 mm to (120.0, 53.9), turned to -90 degrees
- moved R10 76.9 mm to (120.0, 52.0), turned to -90 degrees
- moved C60 59.1 mm to (119.0, 53.9), turned to -90 degrees
- moved C59 59.1 mm to (119.0, 52.0), turned to 90 degrees
- moved C58 53.8 mm to (126.7, 56.1)
- moved C43 45.8 mm to (91.4, 42.1), turned to 0 degrees
- moved C44 45.8 mm to (91.4, 43.2), turned to 0 degrees
- moved C40 45.8 mm to (91.4, 39.1), turned to 0 degrees
- moved C41 45.8 mm to (91.4, 40.1), turned to 0 degrees
- moved C42 45.8 mm to (91.4, 41.1), turned to 0 degrees
- moved C57 38.4 mm to (130.4, 58.6), turned to 0 degrees
- moved C30 37.9 mm to (130.4, 57.6), turned to 0 degrees
- moved C31 37.6 mm to (130.4, 56.6), turned to 0 degrees
- moved C32 37.4 mm to (130.4, 55.6), turned to 0 degrees
- moved C62 37.2 mm to (130.4, 53.6), turned to 0 degrees
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Connections:
- U2 pad E6: /IO/PI8 -> +3V3
Routing:
- net VRAM: track 11.1 -> 131.6 mm, vias 10 -> 25
- net GND: track 2.87 -> 116.3 mm, vias 17 -> 84
- net /Memory/SODT0: track 0.00 -> 18.3 mm, vias 0 -> 3
- net /Memory/SODT1: track 0.00 -> 18.0 mm, vias 0 -> 2
- net /Memory/SCS0: track 0.00 -> 17.9 mm, vias 0 -> 2
- net /Memory/SDQS1P: track 0.00 -> 17.5 mm, vias 0 -> 2
- net /Memory/SDQS1N: track 0.00 -> 17.4 mm, vias 0 -> 2
- net /Memory/SDQ15: track 0.00 -> 17.3 mm, vias 0 -> 3
- net /Memory/SDQ0: track 0.00 -> 17.2 mm, vias 0 -> 1
- net /Memory/SBA0: track 0.00 -> 17.2 mm, vias 0 -> 2
- net /Memory/SDQ2: track 0.00 -> 17.0 mm, vias 0 -> 2
- net /Memory/SCS1: track 0.00 -> 16.8 mm, vias 0 -> 2
- net /Memory/SDQ9: track 0.00 -> 16.8 mm
- net /Memory/SDQ12: track 0.00 -> 16.8 mm, vias 0 -> 3
- net /Memory/SDQ1: track 0.04 -> 16.7 mm, vias 0 -> 3
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- added copper zone on In3.Cu, net +3V3
- added copper zone on In2.Cu, net GND
- added copper zone on In4.Cu, net GND
- removed copper zone on In2.Cu, net +3V3
- removed copper zone on In1.Cu, net VRAM
Other:
- copper layers 4 -> 6

Commit message: project irvine continued
Parts:
- C100, C101, C14, C15, C16, C17, C18, C66, C67, C68, C69, C70, C71, C72, C73, C74, C78, C79, C80, C81, C82, C83, C84, C85, C86, C87, C88, C89, C92, C93, C94, C95, C96, C97, C98, C99, D2, D4, R12, R14, R15, R16, R17, R18, R19, R20, R21, R22, R23, R24, R25, R26, R29, R30, R31, R32, R33, R34, R35, R36, R37, R38, R39, R4, R40, R45, R5, R6, R7, SW1, SW2, Y1, Y2: moved to B.Cu
- moved C77 95.3 mm to (163.9, 52.8), turned to 90 degrees
- moved C16 93.3 mm to (143.2, 54.9)
- moved C76 93.3 mm to (162.8, 52.8), turned to 90 degrees
- moved C75 91.1 mm to (161.3, 52.3), turned to 180 degrees
- moved C14 84.0 mm to (136.4, 57.4)
- moved C15 82.9 mm to (137.9, 61.9), turned to -90 degrees
- moved R28 77.4 mm to (153.5, 57.0)
- moved J1 65.6 mm to (149.1, 68.7), turned to 90 degrees
- moved R6 64.9 mm to (137.6, 55.9), turned to 45 degrees
- moved C67 64.3 mm to (149.9, 105.1), turned to 180 degrees
- moved C68 64.3 mm to (149.9, 107.1), turned to 180 degrees
- moved C69 64.3 mm to (149.9, 109.0), turned to 180 degrees
- moved C70 64.3 mm to (149.9, 111.0), turned to 180 degrees
- moved C71 64.3 mm to (149.9, 113.0), turned to 180 degrees
- moved C72 64.3 mm to (149.9, 115.0), turned to 180 degrees
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Connections:
- U2 pad E6: +3V3 -> /IO/PI8
- U2 pad L14: VRAM -> +1V8
Routing:
- net VBUS: track 2.44 -> 169.7 mm, vias 4 -> 10
- net +1V8: track 5.09 -> 75.7 mm, vias 4 -> 6
- net /IO/NAND_D5: track 1.10 -> 23.1 mm, vias 1 -> 2
- net /Miscellaneous/HDMI_1N: track 0.11 -> 20.7 mm
- net /Miscellaneous/HDMI_CN: track 0.13 -> 20.8 mm
- net /Miscellaneous/HDMI_0N: track 0.15 -> 20.8 mm
- net /Miscellaneous/HDMI_CP: track 0.42 -> 20.8 mm
- net /IO/NAND_D7: track 2.71 -> 23.0 mm
- net /Miscellaneous/HSDA: track 0.00 -> 17.7 mm
- net /Miscellaneous/HSCL: track 0.85 -> 18.2 mm, vias 1 -> 0
- net VHDMI: track 0.00 -> 16.7 mm
- net /Miscellaneous/HDMI_2N: track 4.02 -> 20.7 mm
- net VRAM: track 131.6 -> 148.2 mm, vias 25 -> 24
- net /Miscellaneous/HDMI_1P: track 4.47 -> 20.7 mm
- net /IO/NAND_DS: track 14.1 -> 30.3 mm, vias 2 -> 3
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