File: Radianite-ProjectLemonIrvine/Radianite-ProjectLemonIrvine.kicad_pcb (KiCad board)
At the start: 6 copper layers, 85 x 56 mm, 185 parts, among them J1 FAN, J2 Micro_SD_Card_Det2, J3 Conn_02x20_Odd_Even, J4 RJ45_Abracon_ARJP11A-MASA-B-A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, J5 USB_C_Receptacle_USB2.0_16P, J6 USB_A_Stacked, J7 USB_A_Stacked, J8 AudioJack4, J9 HDMI_A, SW1 434133025816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

Commit message: additions to project irvine
Parts:
- moved C80 68.7 mm to (137.3, 48.9), turned to 90 degrees
Routing:
- net +3V3: track 38.8 -> 40.1 mm, vias 16 -> 17
