File: Radianite-ProjectLemonIrvine/memory.kicad_sch (KiCad schematic)
At the start: 44 parts

Commit message: project irvine continued
Connections:
- net VRAM: no longer U2.L14 (VDD18_DRAM)
- new net +1V8: U2.L14 (VDD18_DRAM)
Changed lines of the file:
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@@
 	)
 	(junction
-		(at 132.08 166.37)
-		(diameter 0)
-		(color 0 0 0 0)
-	)
-	(junction
 		(at 200.66 109.22)
 		(diameter 0)
@@
 	(wire
 		(pts
-			(xy 132.08 166.37) (xy 132.08 168.91)
-		)
-		(stroke
-			(width 0)
-			(type default)
-		)
-	)
-	(wire
-		(pts
 			(xy 78.74 156.21) (xy 93.98 156.21)
 		)
@@
 					(unit 1)
 				)
+			)
+		)
+	)
+	(symbol
+		(lib_id "power:+1V8")
+		(at 132.08 168.91 270)
+		(unit 1)
+		(exclude_from_sim no)
+		(in_bom yes)
+		(on_board yes)
+		(dnp no)
+		(fields_autoplaced yes)
+		(property "Reference" "#PWR0112"
+			(at 128.27 168.91 0)
+			(effects
+				(font
+					(size 1.27 1.27)
+				)
+				(hide yes)
+			)
+		)
+		(property "Value" "+1V8"
+			(at 135.89 168.9099 90)
+			(effects
+				(font
+					(size 1.27 1.27)
+				)
+				(justify left)
+			)
+		)
+		(property "Footprint" ""
+			(at 132.08 168.91 0)
+			(effects
+				(font
+					(size 1.27 1.27)
+				)
+				(hide yes)
+			)
+		)
+		(property "Datasheet" ""
+			(at 132.08 168.91 0)
+			(effects
+				(font
+					(size 1.27 1.27)
+				)
+				(hide yes)
+			)
+		)
+		(property "Description" "Power symbol creates a global label with name \"+1V8\""
+			(at 132.08 168.91 0)
+			(effects
+				(font
+					(size 1.27 1.27)
+				)
+				(hide yes)
+			)
+		)
+		(pin "1"
+		)
+		(instances
+			(project "Radianite-ProjectLemonIrvine"
+				(path "/a0cc354a-60ab-464a-9a28-4a35e48053b0/c3594ab5-3560-48b1-9609-6ea6028d0d19"
+					(reference "#PWR0112")
+					(unit 1)
+				)
