File: Radianite-ProjectLemonIrvine/io.kicad_sch (KiCad schematic)
At the start: 44 parts, among them J2 Micro_SD_Card_Det2, J3 Conn_02x20_Odd_Even, Y1 40MHz

Commit message: few changes
Parts:
- C66: footprint Capacitor_SMD:C_0603_1608Metric -> Capacitor_SMD:C_0402_1005Metric
Changed lines of the file:
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@@
 			)
 		)
-		(property "Footprint" "Capacitor_SMD:C_0603_1608Metric"
+		(property "Footprint" "Capacitor_SMD:C_0402_1005Metric"
 			(at 262.5852 203.2 0)
 			(effects
