File: Radianite-MicroNeo2/Radianite-MicroNeo2.kicad_pcb (KiCad board)
At the start: 4 copper layers, 50 x 33 mm, 87 parts, among them J1 TF-021B-H265, J2 USB_C_Receptacle_USB2.0_16P, J3 USB_C_Receptacle_USB2.0_16P, J4 AudioJack4, J6 Conn_02x16_Odd_Even, SW1 SW_Push, SW2 SW_SPDT, U1 F1C200s, U3 CH340E, U4 W25Q32JVZP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

Commit message: backup
Routing:
- net GND: vias 160 -> 156
Other:
- board text added: "1/3 Partial"
- board text added: "2/3 66% board coverage"
- board text added: "3/3 Full board"
- board text added: "Available expansion board layouts"

Commit message: backup
Parts:
- moved G*** 1.05 mm to (106.5, 65.5)
Other:
- board text removed: "made by the radianite team: zeankun.dev Bobuxstation bgusssssss"
- board text removed: "unleash.the.maker.in.you"
- board text removed: "{dblquote}by far the smallest fully fledged linux computer we ever made from indonesia{dblquote}"

Commit message: 6/3/2025 upstream sync
Parts:
- J1: value TF-021B-H265 -> Micro_SD_Card_Det1
- moved TP6 0.10 mm to (110.6, 72.9)
Connections:
- net /OTG_DM renamed /OTG_D-
- net /OTG_DP renamed /OTG_D+
- net /TTL_DM renamed /TTL_D-
- net /TTL_DP renamed /TTL_D+
- net Net-(U5-XTAL_N) renamed /XTAL-
- net Net-(U5-XTAL_P) renamed /XTAL+
Routing:
- net /OTG_D+: track 26.3 -> 34.3 mm
- net /XTAL+: track 12.0 -> 19.0 mm, vias 0 -> 2
- net /XTAL-: track 13.3 -> 18.0 mm, vias 0 -> 2
- net GND: track 0.00 -> 2.12 mm, vias 156 -> 149
- net VCORE: track 0.00 -> 1.35 mm
- net /SD_CMD: track 34.5 -> 35.8 mm
- net /SD_D3: track 34.7 -> 35.7 mm
- net Net-(U1A-~{RESET}): track 38.5 -> 39.3 mm
- net /SD_D2: track 35.2 -> 35.9 mm
- net /L_FMIN: track 21.3 -> 21.9 mm
- net /OTG_D-: track 35.5 -> 36.1 mm
- net /SD_D0: track 47.7 -> 47.2 mm
