File: Radianite-Novice-RISCV-X/Radianite-Novice-RISCV-X.kicad_pcb (KiCad board)
At the start: 2 copper layers, 68.6 x 53.3 mm, 157 parts, among them J1 USB_C_Receptacle_USB2.0_16P, J2 Conn_01x10_Pin, J3 Conn_01x08_Pin, J4 Conn_01x08, J5 Conn_01x06, J6 Barrel_Jack_Switch, J7 Radianite-Link, SW1 SW_Push, U1 CH32V305RBT6, U2 ESP32-C3-WROOM-02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

Commit message: upstream sync
Parts:
- moved C8 1.77 mm to (103.2, 44.5)
- moved Y1 1.48 mm to (103.6, 47.1)
- moved C7 1.06 mm to (104.0, 49.7)
- moved R1 0.10 mm to (106.9, 46.8)
Routing:
- net Net-(C7-Pad2): track 5.28 -> 4.52 mm
- net /RESET: track 107.8 -> 107.1 mm
- net GND: vias 67 -> 372
Other:
- board text added: "DESIGNED IN INDONESIA JATIM, HOME OF SOUND HOREG"
- board text removed: "DESIGNED IN INDONESIA"

Commit message: add new minor rev
Routing:
- net GND: vias 372 -> 377
Other:
- board text added: "REV 22/11/24 11:00 GMT+7 KICAD 8.0"
- board text removed: "REV 18/10/24 10:57 GMT+7 KICAD 8.0"
