File: Radianite-VariablePortableSSD/Radianite-VariablePortableSSD.kicad_pcb (KiCad board)
At the start: 2 copper layers, 43 x 39 mm, 43 parts, among them J1 USB_C_Receptacle, U1 GL3224, U2 ZDEMDCM064G-95A8, U3 ZDEMDCM064G-95A8, U4 GD25Q32EEIGR, Y1 25MHz

Commit message: backup
Parts:
- moved U4 49.7 mm to (73.8, 52.2), turned to 180 degrees
Changed lines of the file:
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@@
 	(footprint "Package_SON:Winbond_USON-8-1EP_3x2mm_P0.5mm_EP0.2x1.6mm"
 		(layer "F.Cu")
-		(at 24.475 46.255)
+		(at 73.775 52.25 180)
 		(descr "Winbond  USON, 8 Pin (https://www.lcsc.com/datasheet/lcsc_datasheet_2205122030_Winbond-Elec-W25Q16JVUXIQ_C2843335.pdf#page=66f), generated with kicad-footprint-generator ipc_noLead_generator.py")
 		(tags "Winbond USON NoLead")
 		(property "Reference" "U4"
-			(at 0 -1.95 0)
+			(at 0 -1.95 360)
 			(layer "F.SilkS")
 			(effects
@@
 		)
 		(property "Value" "GD25Q32EEIGR"
-			(at 0 1.95 0)
+			(at 0 1.95 360)
 			(layer "F.Fab")
 			(effects
@@
 		)
 		(property "Footprint" "Package_SON:Winbond_USON-8-1EP_3x2mm_P0.5mm_EP0.2x1.6mm"
-			(at 0 0 0)
+			(at 0 0 360)
 			(layer "F.Fab")
 			(hide yes)
@@
 		)
 		(property "Datasheet" "http://www.winbond.com/resource-files/w25q32jv%20revg%2003272018%20plus.pdf"
-			(at 0 0 0)
+			(at 0 0 360)
 			(layer "F.Fab")
 			(hide yes)
@@
 		)
 		(property "Description" "32Mb Serial Flash Memory, Standard/Dual/Quad SPI, DFN-8"
-			(at 0 0 0)
+			(at 0 0 360)
 			(layer "F.Fab")
 			(hide yes)
@@
 		(attr smd)
 		(fp_line
-			(start -1.5 -1.135)
-			(end 1.5 -1.135)
+			(start -1.5 1.135)
+			(end 1.5 1.135)
 			(stroke
 				(width 0.12)
@@
 		)
 		(fp_line
-			(start -1.5 1.135)
-			(end 1.5 1.135)
+			(start -1.5 -1.135)
+			(end 1.5 -1.135)
 			(stroke
 				(width 0.12)
@@
 		)
 		(fp_line
-			(start -2.13 -1.25)
-			(end -2.13 1.25)
+			(start 2.13 1.25)
+			(end 2.13 -1.25)
 			(stroke
 				(width 0.05)
@@
 		)
 		(fp_line
-			(start -2.13 1.25)
-			(end 2.13 1.25)
+			(start 2.13 -1.25)
+			(end -2.13 -1.25)
 			(stroke
 				(width 0.05)
@@
 		)
 		(fp_line
-			(start 2.13 -1.25)
-			(end -2.13 -1.25)
+			(start -2.13 1.25)
+			(end 2.13 1.25)
 			(stroke
 				(width 0.05)
@@
 		)
 		(fp_line
-			(start 2.13 1.25)
-			(end 2.13 -1.25)
+			(start -2.13 -1.25)
+			(end -2.13 1.25)
 			(stroke
 				(width 0.05)
@@
 		)
 		(fp_line
-			(start -1.5 -0.5)
-			(end -1 -1)
+			(start 1.5 1)
+			(end -1.5 1)
 			(stroke
 				(width 0.1)
@@
 		)
 		(fp_line
-			(start -1.5 1)
-			(end -1.5 -0.5)
+			(start 1.5 -1)
+			(end 1.5 1)
 			(stroke
 				(width 0.1)
@@
 		)
 		(fp_line
-			(start 1.5 -1)
-			(end 1.5 1)
+			(start -1.5 1)
+			(end -1.5 -0.5)
 			(stroke
 				(width 0.1)
@@
 		)
 		(fp_line
-			(start 1.5 1)
-			(end -1.5 1)
+			(start -1.5 -0.5)
+			(end -1 -1)
 			(stroke
 				(width 0.1)
@@
 		)
 		(fp_text user "${REFERENCE}"
-			(at 0 0 0)
+			(at 0 0 360)
 			(layer "F.Fab")
 			(effects
@@
 		)
 		(pad "" smd roundrect
-			(at 0 0)
+			(at 0 0 180)
 			(size 0.16 1.29)
 			(layers "F.Paste")
@@
 		)
 		(pad "1" smd roundrect
-			(at -1.425 -0.75)
+			(at -1.425 -0.75 180)
 			(size 0.9 0.25)
 			(layers "F.Cu" "F.Paste" "F.Mask")
@@
 		)
 		(pad "2" smd roundrect
-			(at -1.425 -0.25)
+			(at -1.425 -0.25 180)
 			(size 0.9 0.25)
 			(layers "F.Cu" "F.Paste" "F.Mask")
@@
 		)
 		(pad "3" smd roundrect
-			(at -1.425 0.25)
+			(at -1.425 0.25 180)
 			(size 0.9 0.25)
 			(layers "F.Cu" "F.Paste" "F.Mask")
@@
 		)
 		(pad "4" smd roundrect
-			(at -1.425 0.75)
+			(at -1.425 0.75 180)
 			(size 0.9 0.25)
 			(layers "F.Cu" "F.Paste" "F.Mask")
@@
 		)
 		(pad "5" smd roundrect
-			(at 1.425 0.75)
+			(at 1.425 0.75 180)
 			(size 0.9 0.25)
 			(layers "F.Cu" "F.Paste" "F.Mask")
@@
 		)
 		(pad "6" smd roundrect
-			(at 1.425 0.25)
+			(at 1.425 0.25 180)
 			(size 0.9 0.25)
 			(layers "F.Cu" "F.Paste" "F.Mask")
@@
 		)
 		(pad "7" smd roundrect
-			(at 1.425 -0.25)
+			(at 1.425 -0.25 180)
 			(size 0.9 0.25)
 			(layers "F.Cu" "F.Paste" "F.Mask")
@@
 		)
 		(pad "8" smd roundrect
-			(at 1.425 -0.75)
+			(at 1.425 -0.75 180)
 			(size 0.9 0.25)
 			(layers "F.Cu" "F.Paste" "F.Mask")
@@
 		)
 		(pad "9" smd rect
-			(at 0 0)
+			(at 0 0 180)
 			(size 0.2 1.6)
 			(property pad_prop_heatsink)
@@
 		(height 4)
 		(orientation 1)
-		(gr_text "39,0000 mm"
+		(gr_text "39.0000 mm"
 			(at 102.85 56.5 90)
 			(layer "Dwgs.User")
@@
 		(height 4)
 		(orientation 0)
-		(gr_text "43,0000 mm"
+		(gr_text "43.0000 mm"
 			(at 78.5 78.85 0)
 			(layer "Dwgs.User")

Commit message: 6/3/2025 upstream sync
Parts:
- moved C15 74.3 mm to (95.8, 63.5)
- moved C14 72.5 mm to (95.8, 62.5)
- moved R1 62.5 mm to (79.4, 45.7), turned to 180 degrees
- moved R2 62.3 mm to (79.4, 43.7), turned to 180 degrees
- moved C18 57.6 mm to (79.8, 64.1), turned to 180 degrees
- moved C16 56.8 mm to (77.8, 62.1)
- moved C17 56.3 mm to (77.8, 63.2)
- moved C19 56.3 mm to (79.8, 63.1), turned to 180 degrees
- moved C20 55.1 mm to (79.8, 62.1), turned to 180 degrees
- moved C22 42.8 mm to (61.0, 62.6), turned to 180 degrees
- moved C23 40.6 mm to (61.0, 61.6), turned to 180 degrees
- moved C21 38.1 mm to (61.0, 63.6), turned to 180 degrees
- moved U4 2.29 mm to (75.8, 53.4), turned to 90 degrees
Routing:
- net /EMMC_D4: track 0.00 -> 51.0 mm, vias 0 -> 3
- net /EMMC_D6: track 0.00 -> 50.7 mm, vias 0 -> 3
- net /EMMC_D7: track 0.00 -> 48.3 mm, vias 0 -> 3
- net /EMMC_D2: track 0.00 -> 47.6 mm, vias 0 -> 3
- net /EMMC_D3: track 0.00 -> 45.9 mm, vias 0 -> 3
- net /EMMC_D1: track 0.00 -> 44.7 mm, vias 0 -> 3
- net /EMMC_D0: track 0.00 -> 43.9 mm, vias 0 -> 3
- net SDVCC: track 0.00 -> 31.2 mm, vias 0 -> 4
- net /EMMC_D5: track 0.00 -> 28.0 mm, vias 0 -> 3
- net Net-(J1-CC1): track 0.00 -> 11.7 mm, vias 0 -> 2
- net /FLASH_MISO: track 0.00 -> 11.2 mm
- net Net-(J1-CC2): track 0.00 -> 9.22 mm
- net Net-(U2-VDDI): track 0.00 -> 8.12 mm
- net Net-(U3-VDDI): track 0.00 -> 7.98 mm
- net /FLASH_CS: track 0.00 -> 4.98 mm
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Other:
- copper layers 2 -> 4
